File: Astron.brd (EAGLE design)
At the start: 17.6 x 20 mm, 10 parts, among them J1 CONN_6SCREW_2.54

Commit message: Generated gerbers, minor edits
Other:
- board text added: "Bobby Schulz UMN and NW"
- board text added: "GND"
- board text added: "INT"
- board text added: "Project Astron"
- board text added: "SCL"
- board text added: "SDA"
- board text added: "VBat"
- board text added: "Vcc"
Changed lines of the file:
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@@
 <wire x1="15.125" y1="19.99" x2="2" y2="19.99" width="0" layer="20"/>
 <wire x1="2" y1="19.99" x2="0" y2="17.99" width="0" layer="20" curve="90"/>
+<text x="16.129" y="1.397" size="1.27" layer="21" font="vector" ratio="15" rot="R90">Project
+Astron</text>
+<text x="7.874" y="17.399" size="0.8128" layer="22" font="vector" ratio="15" rot="MR0">Bobby Schulz
+UMN and NW</text>
+<text x="1.27" y="16.256" size="0.8128" layer="22" font="vector" ratio="15" distance="40" rot="MR0" align="center">VBat</text>
+<text x="1.270003125" y="13.716" size="0.8128" layer="22" font="vector" ratio="15" distance="40" rot="MR0" align="center">INT</text>
+<text x="1.27" y="11.176" size="0.8128" layer="22" font="vector" ratio="15" distance="40" rot="MR0" align="center">GND</text>
+<text x="1.27" y="8.636" size="0.8128" layer="22" font="vector" ratio="15" distance="40" rot="MR0" align="center">Vcc</text>
+<text x="1.270003125" y="6.223" size="0.8128" layer="22" font="vector" ratio="15" distance="40" rot="MR0" align="center">SDA</text>
+<text x="1.270003125" y="3.556" size="0.8128" layer="22" font="vector" ratio="15" distance="40" rot="MR0" align="center">SCL</text>
 </plain>
 <attributes>
@@
 <attribute name="MPN" value="BAT-HLD-012-SMT" x="10.922" y="9.906" size="1.778" layer="28" rot="MR270" display="off"/>
 </element>
-<element name="C1" library="bschulz_passives" package="C0603" value="" x="13.081" y="17.399">
+<element name="C1" library="bschulz_passives" package="C0603" value="" x="13.081" y="17.399" smashed="yes">
 <attribute name="DIGIKEY" value="" x="13.081" y="17.399" size="1.778" layer="27" display="off"/>
 <attribute name="MF" value="" x="13.081" y="17.399" size="1.778" layer="27" display="off"/>
 <attribute name="MPN" value="" x="13.081" y="17.399" size="1.778" layer="27" display="off"/>
-</element>
-<element name="C2" library="bschulz_passives" package="C0603" value="" x="10.033" y="17.399" rot="R180">
+<attribute name="VALUE" x="12.446" y="15.494" size="1.27" layer="27"/>
+</element>
+<element name="C2" library="bschulz_passives" package="C0603" value="" x="10.033" y="17.399" smashed="yes" rot="R180">
 <attribute name="DIGIKEY" value="" x="10.033" y="17.399" size="1.778" layer="27" rot="R180" display="off"/>
 <attribute name="MF" value="" x="10.033" y="17.399" size="1.778" layer="27" rot="R180" display="off"/>
 <attribute name="MPN" value="" x="10.033" y="17.399" size="1.778" layer="27" rot="R180" display="off"/>
+<attribute name="VALUE" x="10.668" y="19.304" size="1.27" layer="27" rot="R180"/>
 </element>
 <element name="J1" library="bschulz" package="1X06_SCREW" value="CONN_6SCREW_2.54" x="3.429" y="9.906" smashed="yes" rot="R270">
@@
 <attribute name="MF" value="OnShore" x="3.429" y="9.906" size="1.778" layer="27" rot="R270" display="off"/>
 <attribute name="MPN" value="OSTVN06A150" x="3.429" y="9.906" size="1.778" layer="27" rot="R270" display="off"/>
-<attribute name="NAME" x="14.6812" y="8.3058" size="1.27" layer="25" ratio="10" rot="R90"/>
-</element>
-<element name="U$1" library="bschulz" package="SO08" value="MCP7940SOIC" x="10.287" y="10.414" rot="R180">
+</element>
+<element name="U$1" library="bschulz" package="SO08" value="MCP7940SOIC" x="10.287" y="10.414" smashed="yes" rot="R180">
 <attribute name="DIGIKEY" value="MCP7940N-I/SN-ND" x="10.287" y="10.414" size="1.778" layer="27" rot="R180" display="off"/>
 <attribute name="MF" value="Microchip" x="10.287" y="10.414" size="1.778" layer="27" rot="R180" display="off"/>
@@
 <attribute name="MPN" value="" x="11.557" y="15.367" size="1.778" layer="27" rot="R180" display="off"/>
 </element>
-<element name="C3" library="bschulz_passives" package="C0603" value="0.1uF" x="15.494" y="9.398" rot="R180">
+<element name="C3" library="bschulz_passives" package="C0603" value="0.1uF" x="15.494" y="9.398" smashed="yes" rot="R180">
 <attribute name="DIGIKEY" value="490-6051-1-ND" x="15.494" y="9.398" size="1.778" layer="27" rot="R180" display="off"/>
 <attribute name="MF" value="Murata" x="15.494" y="9.398" size="1.778" layer="27" rot="R180" display="off"/>
 <attribute name="MPN" value="GCM188R71E104KA57D" x="15.494" y="9.398" size="1.778" layer="27" rot="R180" display="off"/>
 </element>
-<element name="C4" library="bschulz_passives" package="C0805" value="10uF" x="15.494" y="11.684" rot="R180">
+<element name="C4" library="bschulz_passives" package="C0805" value="10uF" x="15.494" y="11.684" smashed="yes" rot="R180">
 <attribute name="DIGIKEY" value="490-6473-6-ND" x="15.494" y="11.684" size="1.778" layer="27" rot="R180" display="off"/>
 <attribute name="MF" value="Murata" x="15.494" y="11.684" size="1.778" layer="27" rot="R180" display="off"/>
 <attribute name="MPN" value="GRM21BR61C106KE15K" x="15.494" y="11.684" size="1.778" layer="27" rot="R180" display="off"/>
 </element>
-<element name="R1" library="bschulz_passives" package="R0603" value="10k" x="9.017" y="5.715">
+<element name="R1" library="bschulz_passives" package="R0603" value="10k" x="9.017" y="5.715" smashed="yes">
 <attribute name="DIGIKEY" value="" x="9.017" y="5.715" size="1.778" layer="27" display="off"/>
 <attribute name="MF" value="Yageo" x="9.017" y="5.715" size="1.778" layer="27" display="off"/>
@@
 <attribute name="VALUE_PART" value="" x="9.017" y="5.715" size="1.778" layer="27" display="off"/>
 </element>
-<element name="R2" library="bschulz_passives" package="R0603" value="10k" x="9.017" y="3.556">
+<element name="R2" library="bschulz_passives" package="R0603" value="10k" x="9.017" y="3.556" smashed="yes">
 <attribute name="DIGIKEY" value="" x="9.017" y="3.556" size="1.778" layer="27" display="off"/>
 <attribute name="MF" value="Yageo" x="9.017" y="3.556" size="1.778" layer="27" display="off"/>
@@
 </board>
 </drawing>
+<compatibility>
+<note version="6.3" minversion="6.2.2" severity="warning">
+Since Version 6.2.2 text objects can contain more than one line,
+which will not be processed correctly with this version.
+</note>
+</compatibility>
 </eagle>
