File: Astron.sch (EAGLE design)
At the start: 10 parts, among them J1 CONN_6SCREW_2.54

Commit message: Generated gerbers, minor edits
Connections:
- net GND: now also BT1.-; no longer BT1.BATT-
- net VBAT: now also BT1.+; no longer BT1.BATT+
Changed lines of the file:
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@@
 </segment>
 <segment>
-<pinref part="BT1" gate="G$1" pin="BATT-"/>
+<pinref part="BT1" gate="G$1" pin="-"/>
 <wire x1="63.5" y1="20.32" x2="63.5" y2="17.78" width="0.1524" layer="91"/>
 <pinref part="GND2" gate="1" pin="GND"/>
@@
 </segment>
 <segment>
-<pinref part="BT1" gate="G$1" pin="BATT+"/>
+<pinref part="BT1" gate="G$1" pin="+"/>
 <pinref part="U$1" gate="G$1" pin="VBAT"/>
 <wire x1="63.5" y1="27.94" x2="58.42" y2="27.94" width="0.1524" layer="91"/>
