File: Astron_AltOsc.brd (EAGLE design)
At the start: 17.6 x 20 mm, 10 parts, among them J1 CONN_6SCREW_2.54, U1 MCP7940SOIC

Commit message: Minor updates and added gerber
Parts:
- removed C1, C2: (no value), bschulz_passives:C0603
- removed XTAL1: CRYSTAL3.2X1.5, bschulz:CRYSTAL_3.2X1.5_2-SMD
- added D1: (no value), bschulz:SOT23-3
- added U2: SIT1552, bschulz:LD-4
Connections:
- net GND: now also U2.1, U2.4; no longer C1.2, C2.2
- net N$1: now also U2.2; no longer C1.1, XTAL1.P$1
- net N$2: now also D1.3, U2.3; no longer C2.1, U1.2, XTAL1.P$2
- net VBAT: now also D1.2
- net VCC: now also D1.1
Routing:
- net VBAT: track 41.1 -> 51.1 mm
- net VCC: track 22.1 -> 31.9 mm
- net GND: track 34.0 -> 42.2 mm
- net N$1: track 4.68 -> 1.32 mm
- net N$2: track 4.68 -> 1.62 mm
- removed copper zone on layer 1, net GND
Other:
- board text added: "Project Astron Alt Osc"
- board text removed: "Project Astron"
